File: Xilinx_XC9536XL_EVB.sch (KiCad schematic (older format))
At the start: 54 parts, among them IC1 ATTINY2313-P, P1 CONN_7X2, P2 CONN_2, P3 CONN_3X2, P4 CONN_5, P5 CONN_5, P6 CONN_12, P7 CONN_6, P8 CONN_8, SW1 SW_PUSH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

Commit message: updated footprints libraries (pull-request to official git pending)
Parts:
- C1, C2, C3, C5, C6: footprint (none) -> Capacitors_ThroughHole:C_Rect_L7_W2_P5
- C4: footprint (none) -> Capacitors_ThroughHole:C_Radial_D5_L6_P2.5
- C7, C8: footprint (none) -> Capacitors_ThroughHole:C_Rect_L4_W2.5_P2.5
- D1, D2, D3, D4, D5, D6, D7, D8: footprint (none) -> LEDs:LED-3MM
- IC1: footprint DIL20 -> Sockets_DIP:DIP-20__300; symbol ATTINY2313-P_OLD -> ATTINY2313-P_old
- P1: footprint (none) -> Connect_custom:IDC_Header_Straight_14pins
- P2: footprint (none) -> Connect:bornier2
- P3: footprint (none) -> Pin_Headers:Pin_Header_Straight_2x03
- P4, P5: footprint (none) -> Pin_Headers:Pin_Header_Straight_1x05
- P6: footprint (none) -> Pin_Headers:Pin_Header_Straight_1x12
- P7: footprint (none) -> Pin_Headers:Pin_Header_Straight_1x06
- P8: footprint (none) -> Pin_Headers:Pin_Header_Straight_1x08
- R1, R10, R11, R12, R13, R14, R15, R16, R17, R18, R19, R2, R20, R21, R22, R23, R24, R3, R4, R5, R6, R7, R8, R9: footprint (none) -> Resistors_ThroughHole_custom:Resistor_Horizontal_RM7mm
- RR1: footprint (none) -> Resistors_ThroughHole_custom:Resistor_Array_SIP8
- SW1: footprint (none) -> Buttons_Switches_ThroughHole:SW_PUSH_SMALL
- SW2: footprint (none) -> Buttons_Switches_ThroughHole:SW_DIP_x8_Slide
- U1: footprint (none) -> Sockets:PLCC44
- X1: footprint (none) -> Crystals:Crystal_HC48-U_Vertical

Commit message: updated pcb with new footprints + removed old files
Parts:
- X1: footprint Crystals:Crystal_HC48-U_Vertical -> Crystals:Crystal_HC49-U_Vertical
Changed lines of the file:
@@
 EESchema Schematic File Version 2
-LIBS:Xilinx_XC9536XL_EVB-rescue
 LIBS:power
 LIBS:device
@@
 F 0 "X1" H 2375 3500 60  0000 C CNN
 F 1 "XTAL" H 2300 3200 60  0001 C CNN
-F 2 "Crystals:Crystal_HC48-U_Vertical" H 2200 3350 60  0001 C CNN
+F 2 "Crystals:Crystal_HC49-U_Vertical" H 2200 3350 60  0001 C CNN
 F 3 "" H 2200 3350 60  0001 C CNN
 	1    2200 3350

Commit message: even more clean up
Connections:
- wire segments 207 -> 252
Other:
- moved on the sheet: C5, P1, R11, R12, R13

Commit message: added 3.3v linear regulator
Parts:
- added C9: 10uF, Capacitors_ThroughHole:C_Radial_D5_L6_P2.5, symbol CP1
- added U2: SPX2920T-3.3, TO_SOT_Packages_SMD:TO-252-2Lead, symbol SPX2920T-3.3
Connections:
- net labels added: VCC
- wire segments 252 -> 213
Other:
- note added: "VC"
- note removed: "3.3V"
Changed lines of the file:
@@
 EESchema Schematic File Version 2
+LIBS:regul
+LIBS:power
 LIBS:Xilinx_XC9536XL_EVB-cache
 EELAYER 25 0
@@
 0V
 Text Notes 10350 1150 0    60   ~ 0
-3.3V
+VC
 Text Notes 10300 750  0    60   ~ 0
 Power In
@@
 Connection ~ 9850 1100
 Wire Wire Line
-	6150 7250 6150 7150
-Wire Wire Line
-	6150 7150 6150 7050
-Wire Wire Line
-	6150 7050 6150 6950
-Wire Wire Line
-	6150 6950 6150 6850
-Wire Wire Line
-	6150 6850 6150 6750
-Wire Wire Line
-	6150 6750 6150 6650
-Wire Wire Line
-	6150 6650 6150 6550
+	6150 6550 6150 7250
 Wire Wire Line
 	10150 3050 10150 3300
@@
 Connection ~ 3850 3550
 Wire Wire Line
-	3850 3450 3850 3550
-Wire Wire Line
-	3850 3550 3850 3700
+	3850 3450 3850 3700
 Wire Wire Line
 	1750 2550 1400 2550
@@
 	4400 2600 4400 2100
 Wire Wire Line
-	4400 2100 3600 2100
-Wire Wire Line
-	3600 2100 3150 2100
+	4400 2100 3150 2100
 Wire Wire Line
 	5050 2100 5400 2100
@@
 Connection ~ 2550 3350
 Wire Wire Line
-	2550 3600 2550 3350
-Wire Wire Line
-	2550 3350 2550 3100
+	2550 3100 2550 3600
 Wire Wire Line
 	2550 3100 2450 3100
@@
 Connection ~ 8600 5450
 Wire Wire Line
-	8600 6250 8600 6050
-Wire Wire Line
-	8600 6050 8600 5950
-Wire Wire Line
-	8600 5950 8600 5850
-Wire Wire Line
-	8600 5850 8600 5750
-Wire Wire Line
-	8600 5750 8600 5650
-Wire Wire Line
-	8600 5650 8600 5550
-Wire Wire Line
-	8600 5550 8600 5450
+	8600 5450 8600 6250
 Wire Wire Line
 	9400 5850 9750 5850
@@
 Connection ~ 9400 4900
 Wire Wire Line
-	6450 4900 6550 4900
-Wire Wire Line
-	6550 4900 6650 4900
+	6450 4900 6650 4900
 Connection ~ 6550 4900
 Wire Wire Line
@@
 Connection ~ 7300 1050
 Wire Wire Line
-	6600 1050 6950 1050
-Wire Wire Line
-	6950 1050 7300 1050
-Wire Wire Line
-	7300 1050 7650 1050
-Wire Wire Line
-	7650 1050 8050 1050
-Wire Wire Line
-	8050 1050 8350 1050
+	6600 1050 8350 1050
 Wire Wire Line
 	8350 1050 8350 900
 Connection ~ 8050 1050
 Wire Wire Line
-	6500 1700 6600 1700
-Wire Wire Line
-	6600 1700 6700 1700
+	6500 1700 6700 1700
 Connection ~ 6600 1700
 Wire Wire Line
@@
 	10250 5850 10600 5850
 Wire Wire Line
-	2200 3100 2200 3350
-Wire Wire Line
-	2200 3350 2200 3600
+	2200 3100 2200 3600
 Connection ~ 2200 3350
 Wire Wire Line
 	2200 4000 2200 4100
 Wire Wire Line
-	2200 4100 2375 4100
-Wire Wire Line
-	2375 4100 2550 4100
+	2200 4100 2550 4100
 Wire Wire Line
 	2550 4100 2550 4000
@@
 	2800 3100 2800 3350
 Wire Wire Line
-	1300 1000 1600 1000
-Wire Wire Line
-	1600 1000 2450 1000
+	1300 1000 2450 1000
 Wire Wire Line
 	1300 1000 1300 1050
@@
 Connection ~ 1600 1800
 Wire Wire Line
-	3150 1800 3750 1800
-Wire Wire Line
-	3750 1800 4700 1800
+	3150 1800 4700 1800
 Wire Wire Line
 	4700 1800 4700 2300
@@
 	4700 2300 5400 2300
 Wire Wire Line
-	3150 1900 3700 1900
-Wire Wire Line
-	3700 1900 4600 1900
+	3150 1900 4600 1900
 Wire Wire Line
 	4600 1900 4600 2400
@@
 	4600 2400 5400 2400
 Wire Wire Line
-	3150 2000 3650 2000
-Wire Wire Line
-	3650 2000 4500 2000
+	3150 2000 4500 2000
 Wire Wire Line
 	4500 2000 4500 2500
@@
 	1100 2050 1750 2050
 Wire Wire Line
-	1750 1800 1600 1800
-Wire Wire Line
-	1600 1800 1200 1800
+	1200 1800 1750 1800
 Wire Wire Line
 	1200 1800 1200 1650
@@
 	1200 1650 1000 1650
 Wire Wire Line
-	9400 5450 9400 4900
-Wire Wire Line
-	9400 4900 9400 4600
+	9400 4600 9400 5450
 Wire Wire Line
 	5400 6650 5600 6650
@@
 Connection ~ 6150 6750
 Wire Wire Line
-	1800 6550 2050 6550
-Wire Wire Line
-	2050 6550 2950 6550
-Wire Wire Line
-	1800 6650 2150 6650
-Wire Wire Line
-	2150 6650 2950 6650
-Wire Wire Line
-	1800 6750 2250 6750
-Wire Wire Line
-	2250 6750 2950 6750
-Wire Wire Line
-	1800 6850 2350 6850
-Wire Wire Line
-	2350 6850 2950 6850
-Wire Wire Line
-	1800 6950 2450 6950
-Wire Wire Line
-	2450 6950 2950 6950
-Wire Wire Line
-	2950 7050 2550 7050
-Wire Wire Line
-	2550 7050 1800 7050
-Wire Wire Line
-	2950 7150 2650 7150
-Wire Wire Line
-	2650 7150 1800 7150
-Wire Wire Line
-	2950 7250 2750 7250
-Wire Wire Line
-	2750 7250 1800 7250
+	1800 6550 2950 6550
+Wire Wire Line
+	1800 6650 2950 6650
+Wire Wire Line
+	1800 6750 2950 6750
+Wire Wire Line
+	1800 6850 2950 6850
+Wire Wire Line
+	1800 6950 2950 6950
+Wire Wire Line
+	1800 7050 2950 7050
+Wire Wire Line
+	1800 7150 2950 7150
+Wire Wire Line
+	1800 7250 2950 7250
 Wire Wire Line
 	2150 6400 2150 6650
@@
 	3650 6550 3800 6550
 Wire Wire Line
-	3800 6550 3800 6650
-Wire Wire Line
-	3800 6650 3800 6750
-Wire Wire Line
-	3800 6750 3800 6850
-Wire Wire Line
-	3800 6850 3800 6950
-Wire Wire Line
-	3800 6950 3800 7050
-Wire Wire Line
-	3800 7050 3800 7150
-Wire Wire Line
-	3800 7150 3800 7250
-Wire Wire Line
-	3800 7250 3800 7350
+	3800 6550 3800 7350
 Wire Wire Line
 	3800 6750 3650 6750
@@
 Connection ~ 4850 1550
 Wire Wire Line
-	4750 1550 4850 1550
-Wire Wire Line
-	4850 1550 5000 1550
+	4750 1550 5000 1550
 Wire Wire Line
 	1300 6550 800  6550
@@
 L +3.3V #PWR020
 U 1 1 4D5E3929
-P 9600 900
-F 0 "#PWR020" H 9600 860 30  0001 C CNN
-F 1 "+3.3V" H 9600 1010 30  0000 C CNN
-F 2 "" H 9600 900 60  0001 C CNN
-F 3 "" H 9600 900 60  0001 C CNN
-	1    9600 900
+P 5350 4350
+F 0 "#PWR020" H 5350 4310 30  0001 C CNN
+F 1 "+3.3V" H 5350 4460 30  0000 C CNN
+F 2 "" H 5350 4350 60  0001 C CNN
+F 3 "" H 5350 4350 60  0001 C CNN
+	1    5350 4350
 	1    0    0    -1
 $EndComp
@@
 	1    0    0    -1
 $EndComp
+$Comp
+L GND #PWR030
+U 1 1 56679F04
+P 4850 4950
+F 0 "#PWR030" H 4850 4950 30  0001 C CNN
+F 1 "GND" H 4850 4880 30  0001 C CNN
+F 2 "" H 4850 4950 60  0001 C CNN
+F 3 "" H 4850 4950 60  0001 C CNN
+	1    4850 4950
+	1    0    0    -1
+$EndComp
+$Comp
+L VCC #PWR031
+U 1 1 5667CAF0
+P 9600 900
+F 0 "#PWR031" H 9600 750 50  0001 C CNN
+F 1 "VCC" H 9600 1050 50  0000 C CNN
+F 2 "" H 9600 900 50  0000 C CNN
+F 3 "" H 9600 900 50  0000 C CNN
+	1    9600 900
+	1    0    0    -1
+$EndComp
+$Comp
+L VCC #PWR032
+U 1 1 5667D668
+P 4350 4350
+F 0 "#PWR032" H 4350 4200 50  0001 C CNN
+F 1 "VCC" H 4350 4500 50  0000 C CNN
+F 2 "" H 4350 4350 50  0000 C CNN
+F 3 "" H 4350 4350 50  0000 C CNN
+	1    4350 4350
+	1    0    0    -1
+$EndComp
+Wire Wire Line
+	4350 4350 4350 4450
+Wire Wire Line
+	4350 4450 4450 4450
+Wire Wire Line
+	5250 4450 5350 4450
+Wire Wire Line
+	5350 4450 5350 4350
+Wire Wire Line
+	4850 4750 4850 4950
+Wire Wire Line
+	4350 4850 4850 4850
+$Comp
+L CP1 C9
+U 1 1 5667E437
+P 4350 4650
+F 0 "C9" H 4400 4750 50  0000 L CNN
+F 1 "10uF" H 4400 4550 50  0000 L CNN
+F 2 "Capacitors_ThroughHole:C_Radial_D5_L6_P2.5" H 4350 4650 60  0001 C CNN
+F 3 "" H 4350 4650 60  0001 C CNN
+	1    4350 4650
+	1    0    0    -1
+$EndComp
+Connection ~ 4850 4850
+$Comp
+L SPX2920T-3.3 U2
+U 1 1 56685A35
+P 4850 4500
+F 0 "U2" H 4850 4750 50  0000 C CNN
+F 1 "SPX2920T-3.3" H 4850 4700 50  0000 C CNN
+F 2 "TO_SOT_Packages_SMD:TO-252-2Lead" H 4900 4900 50  0000 C CIN
+F 3 "" H 4850 4500 50  0000 C CNN
+	1    4850 4500
+	1    0    0    -1
+$EndComp
