File: kicad/Xilinx_XC9536XL_EVB.kicad_pcb (KiCad board)
At the start: 2 copper layers, 100 x 66 mm, 60 parts, among them IC1 ATTINY2313-P, P1 CONN_7X2, P2 CONN_2, P3 CONN_3X2, P4 CONN_5, P5 CONN_5, P6 CONN_12, P7 CONN_6, P8 CONN_8, SW1 SW_PUSH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

Commit message: updated pcb with new footprints
Parts:
- C1, C2, C3, C5, C6: footprint Capacitors_ThroughHole:C_Rect_L7_W2_P5 -> Capacitors_THT:C_Rect_L7_W2_P5
- C4, C9: footprint Capacitors_ThroughHole:C_Radial_D5_L6_P2.5 -> Capacitors_THT:C_Radial_D5_L6_P2.5
- C7, C8: footprint Capacitors_ThroughHole:C_Rect_L4_W2.5_P2.5 -> Capacitors_THT:C_Rect_L4_W2.5_P2.5
- IC1: footprint Sockets_DIP:DIP-20__300 -> Housings_DIP:DIP-20_W7.62mm
- P1: footprint Connect:IDC_Header_Straight_14pins -> Connectors:IDC_Header_Straight_14pins
- P2: footprint Connect:bornier2 -> Connectors:bornier2
- R1, R10, R11, R12, R13, R14, R15, R16, R17, R18, R19, R2, R20, R21, R22, R23, R24, R3, R4, R5, R6, R7, R8, R9: footprint Resistors_ThroughHole:Resistor_Horizontal_RM7mm -> Resistors_THT:Resistor_Horizontal_RM7mm
- RR1: footprint Resistors_ThroughHole_custom:Resistor_Array_SIP8 -> Resistors_THT:Resistor_Array_SIP9
- SW1: footprint Buttons_Switches_ThroughHole:SW_PUSH_SMALL -> Buttons_Switches_THT:SW_PUSH_SMALL
- SW2: footprint Buttons_Switches_ThroughHole:SW_DIP_x8_Slide -> Buttons_Switches_THT:SW_DIP_x8_Slide
- moved IC1 12.0 mm to (78.7, 34.3), turned to 270 degrees
- moved RR1 10.2 mm to (114.3, 33.8)
Connections:
- P1 pad 12: Net-(P1-Pad12) -> (no net)
- P1 pad 14: Net-(P1-Pad14) -> (no net)
Routing:
- net +3V3: track 325.9 -> 257.9 mm
- net GND: track 526.3 -> 528.6 mm
- net /RESET: track 53.1 -> 51.3 mm
- net Net-(R14-Pad1): track 34.2 -> 32.4 mm
- added copper zone on B.Cu, net /3V3P
- added copper zone on B.Cu, net Net-(C5-Pad1)
Other:
- net class +3V3 added: clearance 0.254, trace_width 1.016, via_dia 0.889, via_drill 0.635
- net class GND added: clearance 0.254, trace_width 1.016, via_dia 0.889, via_drill 0.635
