File: kicad/Xilinx_XC9536XL_EVB.sch (KiCad schematic (older format))
At the start: 54 parts, among them IC1 ATTINY2313-P, P1 CONN_7X2, P2 CONN_2, P3 CONN_3X2, P4 CONN_5, P5 CONN_5, P6 CONN_12, P7 CONN_6, P8 CONN_8, SW1 SW_PUSH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

Commit message: updated with new libraries/footprints
Parts:
- C1, C2, C3, C5, C6: footprint Capacitors_ThroughHole:C_Rect_L7_W2_P5 -> Capacitors_THT:C_Rect_L7_W2_P5; symbol C -> C-RESCUE-Xilinx_XC9536XL_EVB
- C4: footprint Capacitors_ThroughHole:C_Radial_D5_L6_P2.5 -> Capacitors_THT:C_Radial_D5_L6_P2.5; symbol CP1 -> CP1-RESCUE-Xilinx_XC9536XL_EVB
- C7, C8: footprint Capacitors_ThroughHole:C_Rect_L4_W2.5_P2.5 -> Capacitors_THT:C_Rect_L4_W2.5_P2.5; symbol C -> C-RESCUE-Xilinx_XC9536XL_EVB
- D1, D2, D3, D4, D5, D6, D7, D8: symbol LED -> LED-RESCUE-Xilinx_XC9536XL_EVB
- IC1: footprint Sockets_DIP:DIP-20__300 -> Housings_DIP:DIP-20_W7.62mm
- P1: footprint Connect:IDC_Header_Straight_14pins -> Connectors:IDC_Header_Straight_14pins
- P2: footprint Connect:bornier2 -> Connectors:bornier2
- R1, R10, R11, R12, R13, R14, R15, R16, R17, R18, R19, R2, R20, R21, R22, R23, R24, R3, R4, R5, R6, R7, R8, R9: footprint Resistors_ThroughHole:Resistor_Horizontal_RM7mm -> Resistors_THT:Resistor_Horizontal_RM7mm; symbol R -> R-RESCUE-Xilinx_XC9536XL_EVB
- RR1: footprint Resistors_ThroughHole_custom:Resistor_Array_SIP8 -> Resistors_THT:Resistor_Array_SIP9
- SW2: footprint Buttons_Switches_ThroughHole:SW_DIP_x8_Slide -> Buttons_Switches_THT:SW_DIP_x8_Slide

Commit message: pcb updated with new footprints
Parts:
- SW1: footprint Buttons_Switches_ThroughHole:SW_PUSH_SMALL -> Buttons_Switches_THT:SW_PUSH_SMALL
Changed lines of the file:
@@
 F 0 "SW1" H 5450 1660 50  0000 C CNN
 F 1 "SW_PUSH" H 5300 1470 50  0001 C CNN
-F 2 "Buttons_Switches_ThroughHole:SW_PUSH_SMALL" H 5300 1550 60  0001 C CNN
+F 2 "Buttons_Switches_THT:SW_PUSH_SMALL" H 5300 1550 60  0001 C CNN
 F 3 "" H 5300 1550 60  0001 C CNN
 	1    5300 1550

Commit message: automatic switch to kicad 5 format
Parts:
- C1, C2, C3, C5, C6, C7, C8: symbol C-RESCUE-Xilinx_XC9536XL_EVB -> Xilinx_XC9536XL_EVB-rescue:C-RESCUE-Xilinx_XC9536XL_EVB
- C4: symbol CP1-RESCUE-Xilinx_XC9536XL_EVB -> Xilinx_XC9536XL_EVB-rescue:CP1-RESCUE-Xilinx_XC9536XL_EVB
- D1, D2, D3, D4, D5, D6, D7, D8: symbol LED-RESCUE-Xilinx_XC9536XL_EVB -> Xilinx_XC9536XL_EVB-rescue:LED-RESCUE-Xilinx_XC9536XL_EVB
- IC1: symbol ATTINY2313-P_old -> Xilinx_XC9536XL_EVB-rescue:ATTINY2313-P_old
- P1: symbol CONN_7X2 -> Xilinx_XC9536XL_EVB-rescue:CONN_7X2
- P2: symbol CONN_2 -> Xilinx_XC9536XL_EVB-rescue:CONN_2
- P3: symbol CONN_3X2 -> Xilinx_XC9536XL_EVB-rescue:CONN_3X2
- P4, P5: symbol CONN_5 -> Xilinx_XC9536XL_EVB-rescue:CONN_5
- P6: symbol CONN_12 -> Xilinx_XC9536XL_EVB-rescue:CONN_12
- P7: symbol CONN_6 -> Xilinx_XC9536XL_EVB-rescue:CONN_6
- P8: symbol CONN_8 -> Xilinx_XC9536XL_EVB-rescue:CONN_8
- R1, R10, R11, R12, R13, R14, R15, R16, R17, R18, R19, R2, R20, R21, R22, R23, R24, R3, R4, R5, R6, R7, R8, R9: symbol R-RESCUE-Xilinx_XC9536XL_EVB -> Xilinx_XC9536XL_EVB-rescue:R-RESCUE-Xilinx_XC9536XL_EVB
- RR1: symbol RR8 -> Xilinx_XC9536XL_EVB-rescue:RR8
- SW1: symbol SW_PUSH -> Xilinx_XC9536XL_EVB-rescue:SW_PUSH
- SW2: symbol SW_DIP_8 -> Xilinx_XC9536XL_EVB-rescue:SW_DIP_8
- U1: symbol XC9536PC44 -> Xilinx_XC9536XL_EVB-rescue:XC9536PC44
- X1: symbol XTAL -> Xilinx_XC9536XL_EVB-rescue:XTAL
Connections:
- wire segments 207 -> 252
